File: MC_Telem.kicad_pcb (KiCad board)
At the start: 2 copper layers, 100 x 100 mm, 61 parts, among them J1 Conn_ARM_JTAG_SWD_10, J2 USB_B_Micro, J3 Main Connection, J4 Main Connection, J7 Conn_02x19_Counter_Clockwise, J8 MC Enable, J9 GPS, Q1 Q_NMOS_GDS, Q2 Q_NMOS_GDS, U1 STM32F072RBTx, U2 TPS2113, U3 TCAN1042xV, U4 AMS1117-5.0, U5 TPS5430DDA, U6 MPU-6050, U7 LTC2630, U8 LTC2630, U9 RFD900x

Commit message: Version 2
Parts:
- added C19: 100nF, Capacitor_SMD:C_0402_1005Metric, F.Cu at (140.8, 144.2)
- added C20: 100nF, Capacitor_SMD:C_0402_1005Metric, F.Cu at (137.6, 144.2)
- J7: value Conn_02x19_Counter_Clockwise -> DB37_Male_MountingHoles
- moved C15 7.19 mm to (111.0, 141.9), turned to 180 degrees
- moved C14 5.57 mm to (115.5, 139.8), turned to 90 degrees
- moved R20 4.27 mm to (112.2, 133.2)
- moved C17 3.03 mm to (113.4, 134.7)
- moved U6 2.77 mm to (112.2, 138.1)
- moved R19 2.58 mm to (109.2, 133.2)
- moved C16 0.62 mm to (113.3, 141.4)
Connections:
- J7 pad 0: (no net) -> unconnected-(J7-Pad0)
- J7 pad 2: /Accel- -> /Accel
- J7 pad 21: /Accel -> /Accel-
- U1 pad 55: unconnected-(U1-Pad55) -> /IMU_CS
Routing:
- net /Accel: track 38.1 -> 48.0 mm, vias 1 -> 0
- net /SDA_IMU: track 13.6 -> 16.7 mm
- net /SCL_IMU: track 13.3 -> 16.2 mm
- net Net-(C16-Pad1): track 3.97 -> 1.53 mm
- net +5V: track 185.3 -> 187.6 mm
- net /INT_IMU: track 22.7 -> 24.6 mm
- net +3V3: track 191.1 -> 192.9 mm
- net /CTS: track 45.8 -> 47.6 mm
- net /CAN-: track 145.6 -> 144.9 mm
- net /Rev-: track 16.8 -> 16.2 mm
- net /Indicator+: track 11.6 -> 11.1 mm
- net GND: vias 49 -> 50
Other:
- board text added: "JLCJLCJLCJLC"
- board text added: "Motor Controller Telemetry John Carr Raymond Bernardo Solar Gators V2.0"
- board text removed: "Motor Controller Telemetry John Carr Raymond Bernardo Solar Gators"

Commit message: Adding automation
Parts:
- removed C16, C2: 100nF, Capacitor_SMD:C_0402_1005Metric
- removed C17: 2.2nF, Capacitor_SMD:C_0402_1005Metric
- removed R12: 60, Resistor_SMD:R_0603_1608Metric
- added J5: Conn_01x05, Connector_Wire:SolderWire-0.75sqmm_1x05_P4.8mm_D1.25mm_OD2.3mm, F.Cu at (171.5, 124.5)
- R11: value 60 -> 120; footprint Resistor_SMD:R_0603_1608Metric -> Resistor_SMD:R_1206_3216Metric_Pad1.30x1.75mm_HandSolder
- U6: value MPU-6050 -> LSM6DS3; footprint Sensor_Motion:InvenSense_QFN-24_4x4mm_P0.5mm -> Package_LGA:LGA-14_3x2.5mm_P0.5mm_LayoutBorder3x4y
- moved C15 7.19 mm to (114.2, 135.5), turned to 0 degrees
- moved R11 1.57 mm to (90.0, 96.5), turned to -90 degrees
- moved C14 1.04 mm to (114.6, 139.4)
Connections:
- J7 pad 11: unconnected-(J7-Pad11) -> /MAP_GND
- J7 pad 12: unconnected-(J7-Pad12) -> /MAP_Bit0
- J7 pad 13: unconnected-(J7-Pad13) -> /MAP_Bit2
- J7 pad 31: unconnected-(J7-Pad31) -> /MAP_Bit1
- J7 pad 32: unconnected-(J7-Pad32) -> /MAP_Bit3
- R11 pad 2: Net-(C2-Pad1) -> /CAN+
- U1 pad 27: unconnected-(U1-Pad27) -> /INT2_IMU
- U1 pad 28: /INT_IMU -> /INT1_IMU
- U6 pad 1: GND -> +3V3
- U6 pad 10: Net-(C16-Pad1) -> unconnected-(U6-Pad10)
- U6 pad 11: GND -> unconnected-(U6-Pad11)
- U6 pad 12: /INT_IMU -> +3V3
- U6 pad 13: +3V3 -> /SCL_IMU
- U6 pad 14: (no net) -> /SDA_IMU
- U6 pad 2: (no net) -> +3V3
- U6 pad 3: (no net) -> +3V3
- U6 pad 4: (no net) -> /INT1_IMU
- U6 pad 5: (no net) -> +3V3
- U6 pad 6: unconnected-(U6-Pad6) -> GND
- U6 pad 7: unconnected-(U6-Pad7) -> GND
- U6 pad 9: GND -> /INT2_IMU
Routing:
- net /MAP_GND: track 0.00 -> 71.4 mm
- net /MAP_Bit0: track 0.00 -> 62.3 mm
- net /MAP_Bit1: track 0.00 -> 52.1 mm
- net /MAP_Bit2: track 0.00 -> 37.7 mm
- net /MAP_Bit3: track 0.00 -> 36.4 mm
- net /INT_IMU: track 24.6 -> 0.00 mm, vias 2 -> 0
- net /INT2_IMU: track 0.00 -> 22.1 mm, vias 0 -> 2
- net /INT1_IMU: track 0.00 -> 20.0 mm
- net Net-(C2-Pad1): track 3.00 -> 0.00 mm
- net GND: track 0.00 -> 2.18 mm
- net Net-(C16-Pad1): track 1.53 -> 0.00 mm
- net Net-(C17-Pad1): track 1.45 -> 0.00 mm
- net +3V3: track 192.9 -> 194.3 mm, vias 8 -> 6
- net /SCL_IMU: track 16.2 -> 17.5 mm
- net /SDA_IMU: track 16.7 -> 18.0 mm
