File: MC_Telem.kicad_sch (KiCad schematic)
At the start: 61 parts, among them J1 Conn_ARM_JTAG_SWD_10, J2 USB_B_Micro, J3 Main Connection, J4 Main Connection, J7 Conn_02x19_Counter_Clockwise, J8 MC Enable, J9 GPS, Q1 Q_NMOS_GDS, Q2 Q_NMOS_GDS, U1 STM32F072RBTx, U2 TPS2113, U3 TCAN1042xV, U4 AMS1117-5.0, U5 TPS5430DDA, U6 MPU-6050, U7 LTC2630, U8 LTC2630, U9 RFD900x

Commit message: Version 2
Parts:
- removed J7: Conn_02x19_Counter_Clockwise, Connector_Dsub:DSUB-37_Male_Horizontal_P2.77x2.84mm_EdgePinOffset7.70mm_Housed_MountingHolesOffset9.12mm, symbol Connector_Generic:Conn_02x19_Counter_Clockwise
- added C19, C20: 100nF, Capacitor_SMD:C_0402_1005Metric, symbol Device:C_Small
- added J7: DB37_Male_MountingHoles, Connector_Dsub:DSUB-37_Male_Horizontal_P2.77x2.84mm_EdgePinOffset7.70mm_Housed_MountingHolesOffset9.12mm, symbol Connector:DB37_Male_MountingHoles
- R10, R13, R15, R9: LCSC Part C25197 -> C25804
- R16: LCSC Part C22859 -> C21190
Connections:
- net +5V: now also C19.1, C20.1
- net Accel: now also J7.2
- net Accel+: now also J7.3
- net Accel-: now also J7.21
- net CAN+: now also J7.16
- net CAN-: now also J7.17
- net Eco+: now also J7.5
- net Eco-: now also J7.6
- net GND: now also C19.2, C20.2, J7.28
- net Indicator+: now also J7.15
- net Indicator-: now also J7.14
- net Main+: now also J7.20
- net Main-: now also J7.1
- net Regen: now also J7.22
- net Regen+: now also J7.23
- net Regen-: now also J7.4
- net Rev+: now also J7.7
- net Rev-: now also J7.24
- net IMU_CS: now reaches U1.55 (PB3)
- no-connect marks 73 -> 67
Other:
- moved on the sheet: D1, D2, D5, H1, H2, H3, H4, J1, J8, J9, Q1, Q2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

Commit message: Adding automation
Parts:
- removed C16, C2: 100nF, Capacitor_SMD:C_0402_1005Metric, symbol Device:C_Small
- removed C17: 2.2nF, Capacitor_SMD:C_0402_1005Metric, symbol Device:C_Small
- removed R12: 60, Resistor_SMD:R_0603_1608Metric, symbol Device:R_Small_US
- removed U6: MPU-6050, Sensor_Motion:InvenSense_QFN-24_4x4mm_P0.5mm, symbol Sensor_Motion:MPU-6050
- added J5: Conn_01x05, Connector_Wire:SolderWire-0.75sqmm_1x05_P4.8mm_D1.25mm_OD2.3mm, symbol Connector_Generic:Conn_01x05
- added U6: LSM6DS3, Package_LGA:LGA-14_3x2.5mm_P0.5mm_LayoutBorder3x4y, symbol Sensor_Motion:LSM6DS3
- D1: LCSC Part C34499 -> C2297
- R11: value 60 -> 120; footprint Resistor_SMD:R_0603_1608Metric -> Resistor_SMD:R_1206_3216Metric_Pad1.30x1.75mm_HandSolder
- U4: LCSC Part C347222 -> C6186
Connections:
- net +3V3: now also U6.1 (SDO/SA0), U6.12 (CS), U6.2 (SDX), U6.3 (SCX), U6.5 (VDDIO), U6.8 (VDD)
- net CAN+: now also R11.2
- net GND: now also U6.6 (GND), U6.7 (GND)
- net SCL_IMU: now also U6.13 (SCL)
- net SDA_IMU: now also U6.14 (SDA)
- net INT2_IMU: now reaches U1.27 (PB1)
- net INT2_IMU: now also U6.9 (INT2)
- net MAP_GND: now reaches J7.11
- net MAP_GND: now also J5.1 (Pin_1)
- net MAP_Bit0: now reaches J7.12
- net MAP_Bit0: now also J5.2 (Pin_2)
- net MAP_Bit2: now reaches J7.13
- net MAP_Bit2: now also J5.4 (Pin_4)
- net MAP_Bit1: now reaches J7.31
- net MAP_Bit1: now also J5.3 (Pin_3)
- net MAP_Bit3: now reaches J7.32
- net MAP_Bit3: now also J5.5 (Pin_5)
- net INT_IMU renamed INT1_IMU
- net INT1_IMU: now also U6.4 (INT1)
- no-connect marks 67 -> 64
Other:
- moved on the sheet: R11, R19, R20

Commit message: Fix for automation
Parts:
- C1, C10, C11, C12, C15, C18, C19, C20, C4: LCSC Part C307331 -> (none); LCSC# (none) -> C307331
- C13: LCSC Part C23733 -> (none); LCSC# (none) -> C23733
- C14, C3, C8: LCSC Part C15195 -> (none); LCSC# (none) -> C15195
- C5: LCSC Part C3345 -> (none); LCSC# (none) -> C3345
- C6, C7, C9: LCSC Part C52923 -> (none); LCSC# (none) -> C52923
- D1, D3: LCSC Part C2297 -> (none); LCSC# (none) -> C2297
- D2: LCSC Part C2286 -> (none); LCSC# (none) -> C2286
- D4: LCSC Part C22452 -> (none); LCSC# (none) -> C22452
- D5: LCSC Part C34499 -> (none); LCSC# (none) -> C34499
- L1: LCSC Part C38117 -> (none); LCSC# (none) -> C38117
- Q1, Q2: LCSC Part C20917 -> (none); LCSC# (none) -> C20917
- R1, R2, R3: LCSC Part C8218 -> (none); LCSC# (none) -> C8218
- R10, R13, R15, R9: LCSC Part C25804 -> (none); LCSC# (none) -> C25804
- R14: LCSC Part C22962 -> (none); LCSC# (none) -> C22962
- R16, R18: LCSC Part C21190 -> (none); LCSC# (none) -> C21190
- R17, R19, R20: LCSC Part C4190 -> (none); LCSC# (none) -> C4190
- U4: LCSC Part C6186 -> (none); LCSC# (none) -> C6186
- U5: LCSC Part C9864 -> (none); LCSC# (none) -> C9864
- U6: LCSC Part C784817 -> (none); LCSC# (none) -> C784817
Changed lines of the file:
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@@
       (effects (font (size 1.27 1.27)) hide)
     )
-    (property "LCSC Part" "C2297" (id 4) (at 177.8 80.01 0)
+    (property "LCSC#" "C2297" (id 4) (at 177.8 80.01 0)
       (effects (font (size 1.27 1.27)) hide)
     )
@@
       (effects (font (size 1.27 1.27)) hide)
     )
-    (property "LCSC Part" "C2286" (id 4) (at 177.8 87.63 0)
+    (property "LCSC#" "C2286" (id 4) (at 177.8 87.63 0)
       (effects (font (size 1.27 1.27)) hide)
     )
@@
       (effects (font (size 1.27 1.27)) hide)
     )
-    (property "LCSC Part" "C307331" (id 4) (at 52.07 146.05 0)
+    (property "LCSC#" "C307331" (id 4) (at 52.07 146.05 0)
       (effects (font (size 1.27 1.27)) hide)
     )
@@
       (effects (font (size 1.27 1.27)) hide)
     )
-    (property "LCSC Part" "C9864" (id 4) (at 66.04 177.8 0)
+    (property "LCSC#" "C9864" (id 4) (at 66.04 177.8 0)
       (effects (font (size 1.27 1.27)) hide)
     )
@@
       (effects (font (size 1.27 1.27)) hide)
     )
-    (property "LCSC Part" "C15195" (id 4) (at 83.82 172.72 90)
+    (property "LCSC#" "C15195" (id 4) (at 83.82 172.72 90)
       (effects (font (size 1.27 1.27)) hide)
     )
@@
       (effects (font (size 1.27 1.27)) hide)
     )
-    (property "LCSC Part" "C22452" (id 4) (at 91.44 176.53 90)
+    (property "LCSC#" "C22452" (id 4) (at 91.44 176.53 90)
       (effects (font (size 1.27 1.27)) hide)
     )
@@
       (effects (font (size 1.27 1.27)) hide)
     )
-    (property "LCSC Part" "C38117" (id 4) (at 96.52 172.72 90)
+    (property "LCSC#" "C38117" (id 4) (at 96.52 172.72 90)
       (effects (font (size 1.27 1.27)) hide)
     )
@@
       (effects (font (size 1.27 1.27)) hide)
     )
-    (property "LCSC Part" "C3345" (id 4) (at 101.6 176.53 0)
+    (property "LCSC#" "C3345" (id 4) (at 101.6 176.53 0)
       (effects (font (size 1.27 1.27)) hide)
     )
@@
       (effects (font (size 1.27 1.27)) hide)
     )
-    (property "LCSC Part" "C22962" (id 4) (at 88.9 153.67 0)
+    (property "LCSC#" "C22962" (id 4) (at 88.9 153.67 0)
       (effects (font (size 1.27 1.27)) hide)
     )
@@
       (effects (font (size 1.27 1.27)) hide)
     )
-    (property "LCSC Part" "C25804" (id 4) (at 111.76 176.53 0)
+    (property "LCSC#" "C25804" (id 4) (at 111.76 176.53 0)
       (effects (font (size 1.27 1.27)) hide)
     )
@@
       (effects (font (size 1.27 1.27)) hide)
     )
-    (property "LCSC Part" "C4190" (id 4) (at 111.76 184.15 0)
+    (property "LCSC#" "C4190" (id 4) (at 111.76 184.15 0)
       (effects (font (size 1.27 1.27)) hide)
     )
@@
       (effects (font (size 1.27 1.27)) hide)
     )
-    (property "LCSC Part" "C25804" (id 4) (at 119.38 135.89 0)
+    (property "LCSC#" "C25804" (id 4) (at 119.38 135.89 0)
       (effects (font (size 1.27 1.27)) hide)
     )
@@
       (effects (font (size 1.27 1.27)) hide)
     )
-    (property "LCSC Part" "C307331" (id 4) (at 45.72 176.53 0)
+    (property "LCSC#" "C307331" (id 4) (at 45.72 176.53 0)
       (effects (font (size 1.27 1.27)) hide)
     )
@@
       (effects (font (size 1.27 1.27)) hide)
     )
-    (property "LCSC Part" "C25804" (id 4) (at 149.86 140.97 0)
+    (property "LCSC#" "C25804" (id 4) (at 149.86 140.97 0)
       (effects (font (size 1.27 1.27)) hide)
     )
@@
       (effects (font (size 1.27 1.27)) hide)
     )
-    (property "LCSC Part" "C25804" (id 4) (at 149.86 148.59 0)
+    (property "LCSC#" "C25804" (id 4) (at 149.86 148.59 0)
       (effects (font (size 1.27 1.27)) hide)
     )
@@
       (effects (font (size 1.27 1.27)) hide)
     )
-    (property "LCSC Part" "C6186" (id 4) (at 134.62 173.99 0)
+    (property "LCSC#" "C6186" (id 4) (at 134.62 173.99 0)
       (effects (font (size 1.27 1.27)) hide)
     )
@@
       (effects (font (size 1.27 1.27)) hide)
     )
-    (property "LCSC Part" "C52923" (id 4) (at 123.19 179.07 0)
+    (property "LCSC#" "C52923" (id 4) (at 123.19 179.07 0)
       (effects (font (size 1.27 1.27)) hide)
     )
@@
       (effects (font (size 1.27 1.27)) hide)
     )
-    (property "LCSC Part" "C52923" (id 4) (at 152.4 179.07 0)
+    (property "LCSC#" "C52923" (id 4) (at 152.4 179.07 0)
       (effects (font (size 1.27 1.27)) hide)
     )
@@
       (effects (font (size 1.27 1.27)) hide)
     )
-    (property "LCSC Part" "C21190" (id 4) (at 162.56 177.8 0)
+    (property "LCSC#" "C21190" (id 4) (at 162.56 177.8 0)
       (effects (font (size 1.27 1.27)) hide)
     )
@@
       (effects (font (size 1.27 1.27)) hide)
     )
-    (property "LCSC Part" "C2297" (id 4) (at 158.75 173.99 0)
+    (property "LCSC#" "C2297" (id 4) (at 158.75 173.99 0)
       (effects (font (size 1.27 1.27)) hide)
     )
@@
       (effects (font (size 1.27 1.27)) hide)
     )
-    (property "LCSC Part" "C8218" (id 4) (at 191.77 80.01 90)
+    (property "LCSC#" "C8218" (id 4) (at 191.77 80.01 90)
       (effects (font (size 1.27 1.27)) hide)
     )
@@
       (effects (font (size 1.27 1.27)) hide)
     )
-    (property "LCSC Part" "C8218" (id 4) (at 191.77 87.63 90)
+    (property "LCSC#" "C8218" (id 4) (at 191.77 87.63 90)
       (effects (font (size 1.27 1.27)) hide)
     )
@@
       (effects (font (size 1.27 1.27)) hide)
     )
-    (property "LCSC Part" "C21190" (id 4) (at 111.76 189.23 0)
+    (property "LCSC#" "C21190" (id 4) (at 111.76 189.23 0)
       (effects (font (size 1.27 1.27)) hide)
     )
@@
       (effects (font (size 1.27 1.27)) hide)
     )
-    (property "LCSC Part" "C307331" (id 4) (at 102.87 27.94 0)
+    (property "LCSC#" "C307331" (id 4) (at 102.87 27.94 0)
       (effects (font (size 1.27 1.27)) hide)
     )
@@
       (effects (font (size 1.27 1.27)) hide)
     )
-    (property "LCSC Part" "C307331" (id 4) (at 114.3 27.94 0)
+    (property "LCSC#" "C307331" (id 4) (at 114.3 27.94 0)
       (effects (font (size 1.27 1.27)) hide)
     )
@@
       (effects (font (size 1.27 1.27)) hide)
     )
-    (property "LCSC Part" "C307331" (id 4) (at 125.73 27.94 0)
+    (property "LCSC#" "C307331" (id 4) (at 125.73 27.94 0)
       (effects (font (size 1.27 1.27)) hide)
     )
@@
       (effects (font (size 1.27 1.27)) hide)
     )
-    (property "LCSC Part" "C23733" (id 4) (at 137.16 27.94 0)
+    (property "LCSC#" "C23733" (id 4) (at 137.16 27.94 0)
       (effects (font (size 1.27 1.27)) hide)
     )
@@
       (effects (font (size 1.27 1.27)) hide)
     )
-    (property "LCSC Part" "C15195" (id 4) (at 83.82 27.94 0)
+    (property "LCSC#" "C15195" (id 4) (at 83.82 27.94 0)
       (effects (font (size 1.27 1.27)) hide)
     )
@@
       (effects (font (size 1.27 1.27)) hide)
     )
-    (property "LCSC Part" "C52923" (id 4) (at 93.98 27.94 0)
+    (property "LCSC#" "C52923" (id 4) (at 93.98 27.94 0)
       (effects (font (size 1.27 1.27)) hide)
     )
@@
       (effects (font (size 1.27 1.27)) hide)
     )
-    (property "LCSC Part" "C34499" (id 4) (at 177.8 72.39 0)
+    (property "LCSC#" "C34499" (id 4) (at 177.8 72.39 0)
       (effects (font (size 1.27 1.27)) hide)
     )
@@
       (effects (font (size 1.27 1.27)) hide)
     )
-    (property "LCSC Part" "C8218" (id 4) (at 191.77 72.39 90)
+    (property "LCSC#" "C8218" (id 4) (at 191.77 72.39 90)
       (effects (font (size 1.27 1.27)) hide)
     )
@@
       (effects (font (size 1.27 1.27)) hide)
     )
-    (property "LCSC Part" "C307331" (id 4) (at 50.8 134.62 0)
+    (property "LCSC#" "C307331" (id 4) (at 50.8 134.62 0)
       (effects (font (size 1.27 1.27)) hide)
     )
@@
       (effects (font (size 1.27 1.27)) hide)
     )
-    (property "LCSC Part" "C20917" (id 4) (at 218.44 87.63 0)
+    (property "LCSC#" "C20917" (id 4) (at 218.44 87.63 0)
       (effects (font (size 1.27 1.27)) hide)
     )
@@
       (effects (font (size 1.27 1.27)) hide)
     )
-    (property "LCSC Part" "C20917" (id 4) (at 218.44 73.66 0)
+    (property "LCSC#" "C20917" (id 4) (at 218.44 73.66 0)
       (effects (font (size 1.27 1.27)) hide)
     )
@@
       (effects (font (size 1.27 1.27)) hide)
     )
-    (property "LCSC Part" "C307331" (id 4) (at 213.36 19.05 0)
+    (property "LCSC#" "C307331" (id 4) (at 213.36 19.05 0)
       (effects (font (size 1.27 1.27)) hide)
     )
@@
       (effects (font (size 1.27 1.27)) hide)
     )
-    (property "LCSC Part" "C4190" (id 4) (at 87.63 63.5 0)
+    (property "LCSC#" "C4190" (id 4) (at 87.63 63.5 0)
       (effects (font (size 1.27 1.27)) hide)
     )
@@
       (effects (font (size 1.27 1.27)) hide)
     )
-    (property "LCSC Part" "C15195" (id 4) (at 109.22 48.26 90)
+    (property "LCSC#" "C15195" (id 4) (at 109.22 48.26 90)
       (effects (font (size 1.27 1.27)) hide)
     )
@@
       (effects (font (size 1.27 1.27)) hide)
     )
-    (property "LCSC Part" "C307331" (id 4) (at 247.65 19.05 0)
+    (property "LCSC#" "C307331" (id 4) (at 247.65 19.05 0)
       (effects (font (size 1.27 1.27)) hide)
     )
@@
       (effects (font (size 1.27 1.27)) hide)
     )
-    (property "LCSC Part" "C4190" (id 4) (at 78.74 63.5 0)
+    (property "LCSC#" "C4190" (id 4) (at 78.74 63.5 0)
       (effects (font (size 1.27 1.27)) hide)
     )
@@
       (effects (font (size 1.27 1.27)) hide)
     )
-    (property "LCSC Part" "C784817" (id 4) (at 113.03 66.04 0)
+    (property "LCSC#" "C784817" (id 4) (at 113.03 66.04 0)
       (effects (font (size 1.27 1.27)) hide)
     )
@@
       (effects (font (size 1.27 1.27)) hide)
     )
-    (property "LCSC Part" "C307331" (id 4) (at 119.38 48.26 90)
-      (effects (font (size 1.27 1.27)) hide)
-    )
+    (property "LCSC#" "C307331" (id 4) (at 119.38 48.26 90)
+      (effects (font (size 1.27 1.27)) hide)
+    )
